File: PCB/Display BBM.sch (EAGLE design)
At the start: 9 parts, among them IC1 MEGA8-AI, IC2 7805DT

Commit message: Add Scheme and Layout V 2.0
Haven't place a voltage divider
Parts:
- added X1: (no value), atmel:MISO_MOSIIDC-06V
Connections:
- removed net X1: U1.X1, Y1.2
- removed net X2: U1.X2, Y1.1
- new net N$2: U1.X1, Y1.1
- new net N$3: U1.X2, Y1.2
- net GND: now also X1.GND
- net MISO: now also X1.MISO
- net MOSI: now also X1.MOSI
- net RST: now also X1.!RESET
- net SCK: now also X1.CLK
- net VCC: now also X1.VCC
Other:
- moved on the sheet: Y1
Changed lines of the file:
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@@
 <part name="IC2" library="linear" library_urn="urn:adsk.eagle:library:262" deviceset="78*" device="DT" package3d_urn="urn:adsk.eagle:package:16415/2" technology="05"/>
 <part name="SUPPLY1" library="supply2" library_urn="urn:adsk.eagle:library:372" deviceset="GND" device=""/>
+<part name="X1" library="atmel" deviceset="MISO_MOSI" device="IDC-06V"/>
 </parts>
 <sheets>
@@
 <attribute name="VALUE" x="237.49" y="-33.782" size="1.778" layer="96"/>
 </instance>
-<instance part="Y1" gate="G$1" x="198.12" y="-17.78" smashed="yes" rot="R90" grouprefs="RTC-DS1307">
-<attribute name="NAME" x="195.58" y="-20.32" size="1.27" layer="95" rot="R90"/>
-<attribute name="VALUE" x="201.93" y="-20.32" size="1.27" layer="96" rot="R90"/>
+<instance part="Y1" gate="G$1" x="198.12" y="-17.78" smashed="yes" rot="R270" grouprefs="RTC-DS1307">
+<attribute name="NAME" x="200.66" y="-15.24" size="1.27" layer="95" rot="R270"/>
+<attribute name="VALUE" x="194.31" y="-15.24" size="1.27" layer="96" rot="R270"/>
 </instance>
 <instance part="B1" gate="G$1" x="193.04" y="-25.4" smashed="yes" grouprefs="RTC-DS1307">
@@
 <instance part="SUPPLY1" gate="GND" x="91.44" y="-58.42" smashed="yes">
 <attribute name="VALUE" x="89.535" y="-61.595" size="1.778" layer="96"/>
+</instance>
+<instance part="X1" gate="G$1" x="177.8" y="40.64" smashed="yes" rot="R180">
+<attribute name="NAME" x="184.15" y="32.258" size="1.778" layer="95" rot="R180"/>
 </instance>
 </instances>
@@
 <pinref part="SUPPLY1" gate="GND" pin="GND"/>
 </segment>
+<segment>
+<pinref part="X1" gate="G$1" pin="GND"/>
+<wire x1="170.18" y1="35.56" x2="167.64" y2="35.56" width="0.1524" layer="91"/>
+<label x="167.64" y="35.56" size="0.6096" layer="95" rot="R180" xref="yes"/>
+</segment>
 </net>
 <net name="RST" class="0">
@@
 <label x="88.9" y="53.34" size="0.6096" layer="95" rot="R180" xref="yes" grouprefs="MICRO"/>
 </segment>
+<segment>
+<pinref part="X1" gate="G$1" pin="!RESET"/>
+<wire x1="170.18" y1="38.1" x2="167.64" y2="38.1" width="0.1524" layer="91"/>
+<label x="167.64" y="38.1" size="0.6096" layer="95" rot="R180" xref="yes"/>
+</segment>
 </net>
 <net name="MOSI" class="0">
@@
 <wire x1="139.7" y1="0" x2="142.24" y2="0" width="0.1524" layer="91" grouprefs="MICRO"/>
 <label x="142.24" y="0" size="0.6096" layer="95" xref="yes" grouprefs="MICRO"/>
+</segment>
+<segment>
+<pinref part="X1" gate="G$1" pin="MOSI"/>
+<wire x1="170.18" y1="40.64" x2="167.64" y2="40.64" width="0.1524" layer="91"/>
+<label x="167.64" y="40.64" size="0.6096" layer="95" rot="R180" xref="yes"/>
 </segment>
 </net>
@@
 <label x="248.92" y="-30.48" size="0.6096" layer="95" xref="yes"/>
 </segment>
+<segment>
+<pinref part="X1" gate="G$1" pin="VCC"/>
+<wire x1="170.18" y1="45.72" x2="167.64" y2="45.72" width="0.1524" layer="91"/>
+<label x="167.64" y="45.72" size="0.6096" layer="95" rot="R180" xref="yes"/>
+</segment>
 </net>
 <net name="MISO" class="0">
@@
 <label x="142.24" y="-2.54" size="0.6096" layer="95" xref="yes" grouprefs="MICRO"/>
 </segment>
+<segment>
+<pinref part="X1" gate="G$1" pin="MISO"/>
+<wire x1="170.18" y1="48.26" x2="167.64" y2="48.26" width="0.1524" layer="91"/>
+<label x="167.64" y="48.26" size="0.6096" layer="95" rot="R180" xref="yes"/>
+</segment>
 </net>
 <net name="SCK" class="0">
@@
 <wire x1="139.7" y1="-5.08" x2="142.24" y2="-5.08" width="0.1524" layer="91" grouprefs="MICRO"/>
 <label x="142.24" y="-5.08" size="0.6096" layer="95" xref="yes" grouprefs="MICRO"/>
+</segment>
+<segment>
+<pinref part="X1" gate="G$1" pin="CLK"/>
+<wire x1="170.18" y1="43.18" x2="167.64" y2="43.18" width="0.1524" layer="91"/>
+<label x="167.64" y="43.18" size="0.6096" layer="95" rot="R180" xref="yes"/>
 </segment>
 </net>
@@
 </segment>
 </net>
-<net name="X1" class="0">
-<segment>
-<pinref part="U1" gate="G$1" pin="X1"/>
-<pinref part="Y1" gate="G$1" pin="2"/>
-<wire x1="198.12" y1="-15.24" x2="203.2" y2="-15.24" width="0.1524" layer="91" grouprefs="RTC-DS1307"/>
-</segment>
-</net>
-<net name="X2" class="0">
-<segment>
-<pinref part="U1" gate="G$1" pin="X2"/>
-<pinref part="Y1" gate="G$1" pin="1"/>
-<wire x1="203.2" y1="-20.32" x2="198.12" y2="-20.32" width="0.1524" layer="91" grouprefs="RTC-DS1307"/>
-</segment>
-</net>
 <net name="VBATT" class="0">
 <segment>
@@
 </segment>
 </net>
+<net name="N$2" class="0">
+<segment>
+<pinref part="Y1" gate="G$1" pin="1"/>
+<pinref part="U1" gate="G$1" pin="X1"/>
+<wire x1="198.12" y1="-15.24" x2="203.2" y2="-15.24" width="0.1524" layer="91"/>
+</segment>
+</net>
+<net name="N$3" class="0">
+<segment>
+<pinref part="U1" gate="G$1" pin="X2"/>
+<pinref part="Y1" gate="G$1" pin="2"/>
+<wire x1="203.2" y1="-20.32" x2="198.12" y2="-20.32" width="0.1524" layer="91"/>
+</segment>
+</net>
